File: GPIO_ADC_uHAT.kicad_sch (KiCad schematic)
At the start: 17 parts, among them J1 rpi_uhat_sym, J2 Conn_01x10, J3 Conn_01x10, J4 Conn_01x08, J5 Conn_01x02, U1 MCP23017_SO, U3 CAT24C128, U4 MCP3208

Commit message: made some modifications and added test code
Parts:
- J1: footprint myparts:rpi_uhat_fpt -> myparts:rpi_uhat_fpt_v2
Changed lines of the file:
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@@
 			)
 		)
-		(property "Footprint" "myparts:rpi_uhat_fpt"
+		(property "Footprint" "myparts:rpi_uhat_fpt_v2"
 			(at 144.78 59.69 0)
 			(effects
